File: frogondola_pcb/frogondola.kicad_pcb (KiCad board)
At the start: 2 copper layers, 17.3 x 8.7 mm, 148 parts, among them J1 Conn_01x04_Pin, J10 Conn_01x01_Pin, J2 USB_C_Receptacle_USB2.0_14P, J3 Conn_01x01_Pin, J4 Conn_01x01_Pin, J5 Conn_01x01_Pin, J6 Conn_01x01_Pin, J7 Conn_01x01_Pin, J8 Conn_01x01_Pin, J9 Conn_01x01_Pin, SW1 SW_DPST_x2, SW2 SW_DPST_x2, U1 STM32F072CBTx, U2 TLV74318PDBVR, U3 XC6206PxxxMR, U4 PMW3360DM-T2QU, U5 SRV05-4

Commit message: Adde L60 outline footprint from https://github.com/dededecline/SST60, will update license too.
Parts:
- added H3: PCB Outline, pcb_outline:L60 Outline, F.Cu at (172.6, 78.8)
- H1, H2: moved to F.Cu
- moved U5 177.7 mm to (58.8, 33.0)
- moved R7 171.3 mm to (47.0, 38.5), turned to -90 degrees
- moved R6 168.1 mm to (50.2, 38.5), turned to -90 degrees
- moved U3 163.6 mm to (51.2, 47.8), turned to 90 degrees
- moved F1 159.8 mm to (39.2, 35.2)
- moved R2 156.0 mm to (167.8, 38.5)
- moved R4 156.0 mm to (167.8, 40.5)
- moved R5 153.7 mm to (160.5, 44.2)
- moved SW2 152.8 mm to (198.0, 45.1)
- moved R1 152.1 mm to (193.5, 51.8), turned to -90 degrees
- moved R3 148.1 mm to (160.2, 47.0)
- moved J2 146.4 mm to (48.4, 31.0), turned to 0 degrees
- moved H2 144.3 mm to (188.2, 57.2), turned to 0 degrees
- moved C1 143.5 mm to (193.5, 43.5), turned to -90 degrees
- moved SW1 140.1 mm to (198.0, 52.9)
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Other:
- board size 17.3 x 8.7 mm -> 284.7 x 94.2 mm

Commit message: updated pcb matrix & route.
Parts:
- added S46: MX_stab, PCM_marbastlib-mx:STAB_MX_P_3u, F.Cu at (134.5, 114.4)
- added S50: MX_stab, PCM_marbastlib-mx:STAB_MX_P_3u, F.Cu at (210.7, 114.4)
- moved U3 67.7 mm to (118.8, 52.0), turned to 180 degrees
- moved U1 53.8 mm to (152.1, 40.7), turned to -135 degrees
- moved J3 43.5 mm to (196.2, 76.5)
- moved J4 43.5 mm to (196.2, 80.0)
- moved J10 43.5 mm to (185.6, 80.0)
- moved J5 43.5 mm to (192.7, 76.5)
- moved J6 43.5 mm to (192.7, 80.0)
- moved J7 43.5 mm to (189.1, 76.5)
- moved J8 43.5 mm to (189.1, 80.0)
- moved J9 43.5 mm to (185.6, 76.5)
- moved C11 40.0 mm to (114.4, 53.0), turned to -135 degrees
- moved C12 32.1 mm to (122.3, 53.3), turned to -45 degrees
- moved C10 29.0 mm to (163.1, 60.9)
- moved U2 28.4 mm to (174.6, 42.6), turned to 0 degrees
- moved R2 25.5 mm to (181.3, 60.1), turned to 0 degrees
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Routing:
- net ROW0: track 0.00 -> 336.6 mm
- net ROW1: track 0.00 -> 303.2 mm
- net ROW2: track 0.00 -> 299.3 mm
- net ROW4: track 0.00 -> 260.1 mm
- net ROW3: track 0.00 -> 152.4 mm
- net COL12: track 0.00 -> 81.6 mm
- net COL2: track 0.00 -> 81.6 mm
- net COL1: track 0.00 -> 80.2 mm
- net COL13: track 0.00 -> 78.2 mm
- net COL4: track 0.00 -> 76.7 mm
- net COL10: track 0.00 -> 76.7 mm
- net COL5: track 0.00 -> 74.3 mm
- net COL9: track 0.00 -> 74.3 mm
- net COL14: track 0.00 -> 73.9 mm
- net COL0: track 0.00 -> 72.9 mm
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
Commit message: Routed usb, jst, pmw3360, column matrix.
Parts:
- moved J1 22.0 mm to (65.5, 55.5), turned to -90 degrees
- moved J10 19.2 mm to (167.4, 73.6)
- moved J9 19.2 mm to (167.4, 70.0)
- moved J3 19.2 mm to (178.1, 70.0)
- moved J4 19.2 mm to (178.1, 73.6)
- moved J5 19.2 mm to (174.6, 70.0)
- moved J6 19.2 mm to (174.6, 73.6)
- moved J7 19.2 mm to (171.0, 70.0)
- moved J8 19.2 mm to (171.0, 73.6)
- moved U5 16.4 mm to (49.0, 46.2), turned to 90 degrees
- moved C1 7.96 mm to (194.9, 39.9)
- moved SW2 7.96 mm to (196.0, 35.4)
- moved C11 7.43 mm to (107.0, 53.8)
- moved C12 7.43 mm to (115.0, 54.1)
- moved U3 7.43 mm to (111.4, 52.9)
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Routing:
- net DP: track 0.00 -> 141.5 mm, vias 0 -> 4
- net +3V3: track 53.8 -> 194.8 mm, vias 0 -> 4
- net DN: track 0.00 -> 135.9 mm, vias 0 -> 4
- net COL0: track 72.9 -> 196.7 mm, vias 0 -> 2
- net COL14: track 73.9 -> 189.9 mm, vias 0 -> 2
- net COL1: track 80.2 -> 184.3 mm, vias 0 -> 2
- net +5V: track 3.19 -> 106.6 mm, vias 0 -> 4
- net COL13: track 78.2 -> 172.3 mm, vias 0 -> 2
- net COL2: track 81.6 -> 166.2 mm, vias 0 -> 2
- net COL12: track 81.6 -> 154.4 mm, vias 0 -> 2
- net COL3: track 59.1 -> 121.3 mm, vias 0 -> 2
- net VDD_{1.8V~2.1V}: track 5.33 -> 59.7 mm
- net COL11: track 60.0 -> 110.8 mm, vias 0 -> 2
- net BOOT-1: track 7.60 -> 56.1 mm
- net RST-1: track 7.63 -> 48.7 mm
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
Commit message: Almost done!
Parts:
- C7: value C4_1uF -> C7_1uF
- J10, J7, J8, J9: footprint TestPoint:TestPoint_Pad_1.5x1.5mm -> TestPoint:TestPoint_THTPad_1.5x1.5mm_Drill0.7mm
- R2: value R3_39R -> R2_39R
- R3, R5: value R1_10k -> R3_10k
- R4: value R2_10k -> R4_10k
- R6: value R5_5.1k -> R6_5.1k
- R7: value R6_5.1k -> R7_5.1k
- moved C11 30.1 mm to (77.0, 51.6)
- moved C12 30.1 mm to (84.9, 51.9)
- moved U3 30.1 mm to (81.4, 50.6)
- moved J9 24.4 mm to (187.8, 83.5)
- moved J10 19.5 mm to (184.3, 83.5)
- moved J7 19.5 mm to (187.8, 80.0)
- moved J8 14.7 mm to (184.3, 80.0)
- moved J1 11.4 mm to (56.0, 49.2)
- moved J3 10.2 mm to (187.9, 72.8)
- moved J4 10.2 mm to (187.9, 76.3)
- moved J5 10.2 mm to (184.3, 72.8)
- moved J6 10.2 mm to (184.3, 76.3)
- moved C6 1.27 mm to (159.3, 39.8), turned to 45 degrees
- moved C7 0.92 mm to (177.5, 43.0), turned to 90 degrees
- moved C4 0.07 mm to (145.6, 45.6), turned to -135 degrees
Connections:
- J10 pad 1: ADD7 -> ExMOSI
- J7 pad 1: ADD4 -> ExNSS
- J8 pad 1: ADD5 -> ExSCK
- J9 pad 1: ADD6 -> ExMISO
- U1 pad 10: unconnected-(U1-PA0-Pad10) -> COL9
- U1 pad 11: unconnected-(U1-PA1-Pad11) -> COL8
- U1 pad 12: unconnected-(U1-PA2-Pad12) -> ROW3
- U1 pad 13: unconnected-(U1-PA3-Pad13) -> ROW4
- U1 pad 18: unconnected-(U1-PB0-Pad18) -> ADD2
- U1 pad 19: unconnected-(U1-PB1-Pad19) -> ADD0
- U1 pad 2: unconnected-(U1-PC13-Pad2) -> COL14
- U1 pad 20: unconnected-(U1-PB2-Pad20) -> ADD1
- U1 pad 21: unconnected-(U1-PB10-Pad21) -> ADD3
- U1 pad 25: unconnected-(U1-PB12-Pad25) -> ExNSS
- U1 pad 26: unconnected-(U1-PB13-Pad26) -> ExSCK
- U1 pad 27: unconnected-(U1-PB14-Pad27) -> ExMISO
- U1 pad 28: unconnected-(U1-PB15-Pad28) -> ExMOSI
- U1 pad 29: unconnected-(U1-PA8-Pad29) -> ROW2
- U1 pad 3: unconnected-(U1-PC14-Pad3) -> COL13
- U1 pad 30: unconnected-(U1-PA9-Pad30) -> ROW1
- U1 pad 31: unconnected-(U1-PA10-Pad31) -> ROW0
- U1 pad 34: unconnected-(U1-PA13-Pad34) -> COL7
- U1 pad 37: unconnected-(U1-PA14-Pad37) -> COL6
- U1 pad 38: unconnected-(U1-PA15-Pad38) -> COL5
- U1 pad 39: unconnected-(U1-PB3-Pad39) -> COL4
- U1 pad 4: unconnected-(U1-PC15-Pad4) -> COL12
- U1 pad 40: unconnected-(U1-PB4-Pad40) -> COL3
- U1 pad 41: unconnected-(U1-PB5-Pad41) -> COL2
- U1 pad 42: unconnected-(U1-PB6-Pad42) -> COL1
- U1 pad 43: unconnected-(U1-PB7-Pad43) -> COL0
- U1 pad 5: unconnected-(U1-PF0-Pad5) -> COL11
- U1 pad 6: unconnected-(U1-PF1-Pad6) -> COL10
Routing:
- net ROW4: track 260.1 -> 369.1 mm, vias 0 -> 2
- net ROW3: track 152.4 -> 261.3 mm, vias 0 -> 2
- net COL8: track 45.4 -> 119.4 mm, vias 0 -> 1
- net COL14: track 189.9 -> 261.2 mm, vias 2 -> 3
- net COL13: track 172.3 -> 243.5 mm, vias 2 -> 3
- net COL11: track 110.8 -> 182.0 mm, vias 2 -> 3
- net COL12: track 154.4 -> 225.4 mm, vias 2 -> 3
- net COL10: track 106.9 -> 177.8 mm, vias 2 -> 3
- net COL9: track 83.1 -> 153.7 mm, vias 0 -> 1
- net ExMISO: track 0.00 -> 69.5 mm, vias 0 -> 1
- net ExNSS: track 0.00 -> 68.4 mm, vias 0 -> 1
- net ExMOSI: track 0.00 -> 67.0 mm, vias 0 -> 1
- net ExSCK: track 0.00 -> 65.0 mm, vias 0 -> 1
- net ROW2: track 299.3 -> 361.1 mm, vias 0 -> 2
- net ADD1: track 0.00 -> 54.0 mm, vias 0 -> 2
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- added copper zone on B.Cu, net GND
- added copper zone on F.Cu, net GND
Other:
- board text added: ","
- board text added: "."
- board text added: "/"
- board text added: ";"
- board text added: "A"
- board text added: "Alt"
- board text added: "B"
- board text added: "B0"
- board text added: "B1"
- board text added: "B10"
- board text added: "B2"
- board text added: "Back"
- board text added: "C"
- board text added: "Control"
- board text added: "Ctrl"
- board text added: "D"
- board text added: "Designed by My-Fi"
- board text added: "E"
- board text added: "Enter"
- board text added: "Esc"
- board text added: "F"
- board text added: "G"
- board text added: "H"
- board text added: "I"
- board text added: "J"
- board text added: "K"
- board text added: "L"
- board text added: "M"
- board text added: "Mod"
- board text added: "N"
- board text added: "O"
- board text added: "P"
- board text added: "Q"
- board text added: "R"
- board text added: "S"
- board text added: "SPI2_MISO I2C2_SDA"
- board text added: "SPI2_MOSI"
- board text added: "SPI2_NSS"
- board text added: "SPI2_SCK I2C2_SCL"
- board text added: "Shift"
- board text added: "Super"
- board text added: "T"
- board text added: "U"
- board text added: "V"
- board text added: "W"
- board text added: "X"
- board text added: "Y"
- board text added: "Z"
